Commit message: Human min with hands

File: urdf/human_min.urdf (robot description, URDF)
Before this commit: robot HUMAN, 3 links, 2 joints
Links:
- added link LArmLink, mass 1.96; collision mesh filename=package://human_description/meshes/LArmLinkFull.dae; visual mesh filename=package://human_description/meshes/LArmLinkFull.dae
- added link LElbowLink, mass 0.25; collision mesh filename=package://human_description/meshes/LElbowLink.dae; visual mesh filename=package://human_description/meshes/LElbowLink.dae
- added link LForearmLink, mass 1.18; collision mesh filename=package://human_description/meshes/LForearmLink.dae; visual mesh filename=package://human_description/meshes/LForearmLink.dae
- added link LHandLink, mass 0.272; collision mesh filename=package://human_description/meshes/LWrist.dae; visual mesh filename=package://human_description/meshes/LWrist.dae
- added link RArmLink, mass 1.96; collision mesh filename=package://human_description/meshes/RArmLinkFull.dae; visual mesh filename=package://human_description/meshes/RArmLinkFull.dae
- added link RElbowLink, mass 0.25; collision mesh filename=package://human_description/meshes/RElbowLink.dae; visual mesh filename=package://human_description/meshes/RElbowLink.dae
- added link RForearmLink, mass 1.18; collision mesh filename=package://human_description/meshes/RForearmLink.dae; visual mesh filename=package://human_description/meshes/RForearmLink.dae
- added link RHandLink, mass 0.272; collision mesh filename=package://human_description/meshes/RWrist.dae; visual mesh filename=package://human_description/meshes/RWrist.dae
- added link forearm2lwrist_1, mass 0.05
- added link forearm2rwrist_1, mass 0.05
- added link torso2lshoulder_1, mass 0.2
- added link torso2lshoulder_2, mass 0.2
- added link torso2rshoulder_1, mass 0.2
- added link torso2rshoulder_2, mass 0.2
Joints:
- added joint LArm_0: type revolute, parent TorsoLink, child torso2lshoulder_1, origin xyz=-0.05 0.15 0.35 rpy=0.0 0.0 0.0, axis 1 0 0, limit lower=-1.42 upper=1.57 effort=100 velocity=100
- added joint LArm_1: type revolute, parent torso2lshoulder_1, child torso2lshoulder_2, origin xyz=-0.0 0.0 0.0 rpy=0.0 0.0 0.0, axis 0 1 0, limit lower=-1.2 upper=1.2 effort=100 velocity=100
- added joint LArm_2: type revolute, parent torso2lshoulder_2, child LArmLink, origin xyz=-0.0 0.0 0.0 rpy=0.0 0.0 0.0, axis 0 0 1, limit lower=-2.8 upper=0.9 effort=100 velocity=100
- added joint LElbow: type revolute, parent LArmLink, child LElbowLink, origin xyz=-0.0 0.2 0.0 rpy=0.0 0.0 0.0, axis 0 1 0, limit lower=-1.57 upper=1.0 effort=100 velocity=100
- added joint LForearm: type revolute, parent LElbowLink, child LForearmLink, origin xyz=-0.01 0.05 0.0 rpy=0.0 0.0 0.0, axis 0 0 1, limit lower=-2.5 upper=0.0 effort=100 velocity=100
- added joint LWrist_0: type revolute, parent LForearmLink, child forearm2lwrist_1, origin xyz=0.01 0.24 -0.01 rpy=0.0 0.0 0.0, axis 1 0 0, limit lower=-1.5 upper=1.5 effort=100 velocity=100
- added joint LWrist_1: type revolute, parent forearm2lwrist_1, child LHandLink, origin xyz=0.0 0.0 0.0 rpy=0.0 0.0 0.0, axis 0 0 1, limit lower=-0.35 upper=0.35 effort=100 velocity=100
- added joint RArm_0: type revolute, parent TorsoLink, child torso2rshoulder_1, origin xyz=-0.05 -0.15 0.35 rpy=0.0 0.0 0.0, axis 1 0 0, limit lower=-1.42 upper=1.57 effort=100 velocity=100
- added joint RArm_1: type revolute, parent torso2rshoulder_1, child torso2rshoulder_2, origin xyz=-0.0 0.0 0.0 rpy=0.0 0.0 0.0, axis 0 1 0, limit lower=-1.2 upper=1.2 effort=100 velocity=100
- added joint RArm_2: type revolute, parent torso2rshoulder_2, child RArmLink, origin xyz=-0.0 0.0 0.0 rpy=0.0 0.0 0.0, axis 0 0 1, limit lower=-0.9 upper=2.8 effort=100 velocity=100
- added joint RElbow: type revolute, parent RArmLink, child RElbowLink, origin xyz=-0.0 -0.2 0.0 rpy=0.0 0.0 0.0, axis 0 1 0, limit lower=-1.57 upper=1.0 effort=100 velocity=100
- added joint RForearm: type revolute, parent RElbowLink, child RForearmLink, origin xyz=-0.01 -0.05 0.0 rpy=0.0 0.0 0.0, axis 0 0 1, limit lower=0.0 upper=2.5 effort=100 velocity=100
- added joint RWrist_0: type revolute, parent RForearmLink, child forearm2rwrist_1, origin xyz=0.01 -0.24 -0.01 rpy=0.0 0.0 0.0, axis 1 0 0, limit lower=-1.5 upper=1.5 effort=100 velocity=100
- added joint RWrist_1: type revolute, parent forearm2rwrist_1, child RHandLink, origin xyz=0.0 0.0 0.0 rpy=0.0 0.0 0.0, axis 0 0 1, limit lower=-0.35 upper=0.35 effort=100 velocity=100

Commit message: Added missing torso move joints

File: urdf/human_min.urdf (robot description, URDF)
Before this commit: robot HUMAN, 17 links, 16 joints
Links:
- added link base_link1
- added link base_link2
Joints:
- removed joint base
- added joint T0: type revolute, parent base_link, child base_link1, origin xyz=0.0 0.0 0.0 rpy=0.0 0.0 0.0, axis 1 0 0, limit lower=-3.1457 upper=3.1457 effort=100 velocity=100
- added joint T1: type revolute, parent base_link1, child base_link2, origin xyz=0.0 0.0 0.0 rpy=0.0 0.0 0.0, axis 0 1 0, limit lower=-3.1457 upper=3.1457 effort=100 velocity=100
- added joint T2: type revolute, parent base_link2, child TorsoLink, origin xyz=0.0 0.0 0.0 rpy=0.0 0.0 0.0, axis 0 0 1, limit lower=-3.1457 upper=3.1457 effort=100 velocity=100
